Commit message: Add Gazebo simulation, Nav2 navigation, depth camera, LiDAR scan visualization

File: ros2_ws/interbotix_xslocobot_descriptions/urdf/kobuki_version/locobot_kobuki.urdf.xacro (robot description, xacro)
@@ -465,3 +465,24 @@
     </plugin>
   </gazebo>
+  <link name="$(arg robot_name)/depth_camera_link">
+    <visual><geometry><box size="0.05 0.05 0.05"/></geometry></visual>
+    <inertial><mass value="0.1"/><inertia ixx="0.001" ixy="0" ixz="0" iyy="0.001" iyz="0" izz="0.001"/></inertial>
+  </link>
+  <joint name="depth_camera_joint" type="fixed">
+    <parent link="$(arg robot_name)/base_link"/>
+    <child link="$(arg robot_name)/depth_camera_link"/>
+    <origin xyz="0.1 0 0.4" rpy="0 0 0"/>
+  </joint>
+  <gazebo reference="$(arg robot_name)/depth_camera_link">
+    <sensor name="depth_camera" type="depth_camera">
+      <update_rate>10</update_rate>
+      <topic>/camera/depth</topic>
+      <gz_frame_id>$(arg robot_name)/depth_camera_link</gz_frame_id>
+      <camera>
+        <horizontal_fov>1.047</horizontal_fov>
+        <image><width>320</width><height>240</height></image>
+        <clip><near>0.1</near><far>10.0</far></clip>
+      </camera>
+    </sensor>
+  </gazebo>
 </robot>

File: ros2_ws/interbotix_xslocobot_descriptions/urdf/lidar.urdf.xacro (robot description, xacro)
@@ -63,12 +63,11 @@
     <gazebo reference="$(arg robot_name)/laser_frame_link">
       <material>Custom/Interbotix</material>
-      <sensor type="ray" name="rplidar">
+      <sensor name="rplidar" type="gpu_lidar">
         <pose>0 0 0 0 0 0</pose>
-        <visualize>false</visualize>
-        <update_rate>30</update_rate>
-        <ray>
+        <update_rate>10</update_rate>
+        <lidar>
           <scan>
             <horizontal>
-              <samples>400</samples>
+              <samples>360</samples>
               <resolution>1</resolution>
               <min_angle>-3.14159</min_angle>
@@ -78,5 +77,5 @@
           <range>
             <min>0.2</min>
-            <max>16.0</max>
+            <max>12.0</max>
             <resolution>0.02</resolution>
           </range>
@@ -86,6 +85,5 @@
             <stddev>0.01</stddev>
           </noise>
-        </ray>
-        <!-- ROS1 laser plugin removed for Gazebo Harmonic compatibility -->
+        </lidar>
       </sensor>
     </gazebo>
